File: pcb/FPGA_Config.sch (KiCad schematic (older format))
At the start: 25 parts, among them J901 JTAG-XILINX-TC, SW901 SW_PUSH, U401 XC7Axxt-FGG484, U901 S25FL256SAGNFI

Commit message: Ready for fab
Parts:
- U401: symbol XC7Axxt-FGG484 -> XC7Axxt-FGG484-RESCUE-artix7_pcie_pcb
Changed lines of the file:
@@
 EESchema Schematic File Version 2
+LIBS:artix7_pcie_pcb-rescue
 LIBS:power
 LIBS:device
@@
 LIBS:valves
 LIBS:wbraun_ic_lib
-LIBS:pgmfoot
 LIBS:artix7_pcie_pcb-cache
 EELAYER 25 0
@@
 $EndDescr
 $Comp
-L XC7Axxt-FGG484 U401
+L XC7Axxt-FGG484-RESCUE-artix7_pcie_pcb U401
 U 1 1 56341AFC
 P 1700 4950
@@
 $EndComp
 $Comp
-L XC7Axxt-FGG484 U401
+L XC7Axxt-FGG484-RESCUE-artix7_pcie_pcb U401
 U 2 1 564F5018
 P 4800 4950
