File: pcb/FPGA_gnd.sch (KiCad schematic (older format))
At the start: 1 part, among them U401 XC7Axxt-FGG484

Commit message: Finished most of the routing, removed DDR-3
Parts:
- U401: footprint (none) -> wbraun_smd:BGA_484_22x22_FULLARRAY_1MM
Changed lines of the file:
@@
 $Descr A4 11693 8268
 encoding utf-8
-Sheet 13 13
+Sheet 13 11
 Title ""
 Date ""
@@
 F 0 "U401" H 3600 1650 60  0000 C CNN
 F 1 "XC7Axxt-FGG484" H 3900 6850 60  0000 C CNN
-F 2 "" H 4500 4300 60  0000 C CNN
+F 2 "wbraun_smd:BGA_484_22x22_FULLARRAY_1MM" H 4500 4300 60  0001 C CNN
 F 3 "" H 4500 4300 60  0000 C CNN
 	9    4500 4250
@@
 Connection ~ 3000 6600
 $Comp
-L GND #PWR0172
+L GND #PWR0163
 U 1 1 5665ED49
 P 3000 6900
-F 0 "#PWR0172" H 3000 6650 50  0001 C CNN
+F 0 "#PWR0163" H 3000 6650 50  0001 C CNN
 F 1 "GND" H 3000 6750 50  0000 C CNN
 F 2 "" H 3000 6900 50  0000 C CNN
@@
 $EndComp
 $Comp
-L GND #PWR0173
+L GND #PWR0164
 U 1 1 5665ED60
 P 6000 5800
-F 0 "#PWR0173" H 6000 5550 50  0001 C CNN
+F 0 "#PWR0164" H 6000 5550 50  0001 C CNN
 F 1 "GND" H 6000 5650 50  0000 C CNN
 F 2 "" H 6000 5800 50  0000 C CNN

Commit message: Ready for fab
Parts:
- U401: symbol XC7Axxt-FGG484 -> XC7Axxt-FGG484-RESCUE-artix7_pcie_pcb
Changed lines of the file:
@@
 EESchema Schematic File Version 2
+LIBS:artix7_pcie_pcb-rescue
 LIBS:power
 LIBS:device
@@
 LIBS:valves
 LIBS:wbraun_ic_lib
-LIBS:pgmfoot
 LIBS:artix7_pcie_pcb-cache
 EELAYER 25 0
@@
 $EndDescr
 $Comp
-L XC7Axxt-FGG484 U401
+L XC7Axxt-FGG484-RESCUE-artix7_pcie_pcb U401
 U 9 1 5665CDB7
 P 4500 4250
