File: pcb/User_IO.sch (KiCad schematic (older format))
At the start: 15 parts, among them P1201 CONN_02X05, P1202 CONN_02X05, SW1201 SW_PUSH, SW1202 SW_PUSH, U401 XC7Axxt-FGG484

Commit message: Ready for fab
Parts:
- U401: symbol XC7Axxt-FGG484 -> XC7Axxt-FGG484-RESCUE-artix7_pcie_pcb
Changed lines of the file:
@@
 EESchema Schematic File Version 2
+LIBS:artix7_pcie_pcb-rescue
 LIBS:power
 LIBS:device
@@
 LIBS:valves
 LIBS:wbraun_ic_lib
-LIBS:pgmfoot
 LIBS:artix7_pcie_pcb-cache
 EELAYER 25 0
@@
 $EndDescr
 $Comp
-L XC7Axxt-FGG484 U401
+L XC7Axxt-FGG484-RESCUE-artix7_pcie_pcb U401
 U 5 1 565FC0A5
 P 3400 3950
