File: pcb/artix7_pcie_pcb.kicad_pcb (KiCad board)
At the start: 4 copper layers, 100 x 115.2 mm, 192 parts, among them CON301 BARREL_JACK, J1101 SFP_CONN, J201 PCIe_x1, J801 FX10B-80S/8-SV, J901 JTAG-XILINX-TC, P1201 CONN_02X05, P1202 CONN_02X05, SW1201 SW_PUSH, SW1202 SW_PUSH, SW901 SW_PUSH, U1001 FOX924, U1002 NB3L553, U1003 Si5338C, U301 LTM4622, U302 LTM4622, U303 ADP170, U401 XC7Axxt-FGG484, U901 S25FL256SAGNFI

Commit message: power routing finished
Parts:
- C313, C314: footprint wbraun_smd:0402_in_grid -> wbraun_smd:C_0402
- C404, C424, C427, C452, C460, C464, C468, C471, C475: moved to F.Cu
- C411, C417, C418, C419, C423, C425, C428, C430, C433, C435, C438, C439, C440, C454, C458, C459, C462, C463, C466, C467, C469, C470, C473: moved to B.Cu
- R304: value 13.3K -> 8.25K
- R308: value 8.25K -> 13.3K
- moved C470 137.2 mm to (99.8, 82.8), turned to 0 degrees
- moved C438 135.6 mm to (104.0, 84.0), turned to 0 degrees
- moved C423 135.6 mm to (101.0, 85.0), turned to 0 degrees
- moved C433 131.4 mm to (107.0, 83.0), turned to 0 degrees
- moved C454 130.5 mm to (103.0, 81.0), turned to 0 degrees
- moved C462 129.5 mm to (106.0, 80.0), turned to 0 degrees
- moved C440 122.6 mm to (113.0, 83.0), turned to 180 degrees
- moved C419 120.3 mm to (103.0, 86.0), turned to 180 degrees
- moved C466 120.0 mm to (117.0, 80.0), turned to 0 degrees
- moved C418 118.8 mm to (110.0, 98.0), turned to 180 degrees
- moved C428 113.8 mm to (105.0, 98.0), turned to 0 degrees
- moved C458 113.4 mm to (107.0, 84.5), turned to 0 degrees
- moved C434 112.7 mm to (101.0, 80.0), turned to 180 degrees
- moved C417 110.0 mm to (109.5, 84.0)
- moved C429 109.8 mm to (108.0, 97.0), turned to 0 degrees
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Connections:
- C308 pad 1: +3V3 -> +5V
- C309 pad 1: +5V -> +3V3
- C310 pad 1: +3V3 -> +5V
- C311 pad 1: +5V -> +3V3
- U302 pad A1: +5V -> +3V3
- U302 pad B1: +5V -> +3V3
- U302 pad D1: +3V3 -> +5V
- U302 pad E1: +3V3 -> +5V
Routing:
- net GND: track 185.2 -> 310.4 mm, vias 178 -> 240
- net +3V3: track 66.5 -> 124.8 mm, vias 61 -> 80
- net /FPGA Config/DONE: track 20.7 -> 58.7 mm, vias 0 -> 2
- net /FPGA Config/M2: track 7.81 -> 25.5 mm, vias 0 -> 2
- net /FPGA Config/M0: track 9.11 -> 26.1 mm
- net /FPGA Config/INIT_B: track 9.26 -> 24.6 mm
- net /FPGA Config/M1: track 11.2 -> 25.3 mm, vias 1 -> 2
- net /FPGA Config/TCK: track 18.7 -> 32.1 mm
- net +1V8: track 37.2 -> 48.8 mm, vias 9 -> 16
- net /FPGA Config/TDO: track 14.5 -> 25.1 mm, vias 1 -> 2
- net /FPGA Config/PROGRAM_B: track 33.4 -> 43.8 mm, vias 1 -> 2
- net /FPGA Config/TDI: track 25.2 -> 35.2 mm, vias 1 -> 2
- net /FPGA Config/TMS: track 16.5 -> 24.9 mm, vias 1 -> 2
- net +1V0: track 50.6 -> 57.8 mm, vias 22 -> 31
- net +1V2: track 0.00 -> 6.08 mm
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
Commit message: routing finished, need final check
Parts:
- removed TP201, TP202: Test_Pad, Wire_Pads:SolderWirePad_single_0-8mmDrill
- C464, C468, C471, C475: moved to B.Cu
- R1208: moved to F.Cu
- moved J201 179.5 mm to (99.0, 151.0)
- moved C468 32.4 mm to (96.0, 78.2)
- moved C471 31.0 mm to (96.0, 81.0)
- moved C475 29.3 mm to (97.5, 78.2)
- moved C464 28.9 mm to (97.5, 81.0)
- moved SW1202 25.8 mm to (113.8, 125.8), turned to 0 degrees
- moved R201 25.1 mm to (108.0, 112.0), turned to 270 degrees
- moved C424 23.5 mm to (128.5, 73.0), turned to 0 degrees
- moved P1201 22.3 mm to (137.0, 100.8), turned to 0 degrees
- moved D1201 20.4 mm to (111.2, 115.8), turned to 90 degrees
- moved C460 20.4 mm to (124.5, 73.0), turned to 0 degrees
- moved P1202 20.2 mm to (137.0, 119.0), turned to 0 degrees
- moved R1201 16.1 mm to (111.2, 112.0), turned to 90 degrees
- moved D1202 15.9 mm to (114.2, 115.8), turned to 90 degrees
- moved SW1201 14.3 mm to (123.8, 125.8), turned to 0 degrees
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Connections:
- J201 pad B17: /PCIe Connector/PCIE_PRSNT#2 -> /PCIe Connector/PCIE_PRSNT#1
- R201 pad 1: /PCIe Connector/PERST# -> /User IO/PCIE_PERST
- U401 pad AA1: Net-(U401-PadAA1) -> /User IO/IO11
- U401 pad AA3: /User IO/IO1 -> /User IO/IO5
- U401 pad AA4: /User IO/IO5 -> /User IO/IO1
- U401 pad AA5: /User IO/IO2 -> Net-(U401-PadAA5)
- U401 pad AB1: Net-(U401-PadAB1) -> /User IO/IO10
- U401 pad AB2: Net-(U401-PadAB2) -> /User IO/IO7
- U401 pad AB3: Net-(U401-PadAB3) -> /User IO/IO4
- U401 pad AB5: /User IO/IO3 -> Net-(U401-PadAB5)
- U401 pad R2: /User IO/B0 -> Net-(U401-PadR2)
- U401 pad R3: Net-(U401-PadR3) -> /User IO/IO9
- U401 pad R6: Net-(U401-PadR6) -> /User IO/PCIE_PERST
- U401 pad T1: /User IO/LED1 -> /User IO/B0
- U401 pad T3: /User IO/LED0 -> Net-(U401-PadT3)
- U401 pad T4: /User IO/IO9 -> Net-(U401-PadT4)
- U401 pad T5: /User IO/IO10 -> Net-(U401-PadT5)
- U401 pad U1: /User IO/LED2 -> /User IO/B1
- U401 pad U2: /User IO/LED3 -> /User IO/LED0
- U401 pad U3: Net-(U401-PadU3) -> /User IO/LED2
- U401 pad U5: /User IO/IO11 -> Net-(U401-PadU5)
- U401 pad U6: /User IO/IO14 -> Net-(U401-PadU6)
- U401 pad V2: Net-(U401-PadV2) -> /User IO/LED1
- U401 pad V3: Net-(U401-PadV3) -> /User IO/LED3
- U401 pad V4: /User IO/IO6 -> /User IO/IO0
- U401 pad V5: /User IO/IO15 -> Net-(U401-PadV5)
- U401 pad W1: Net-(U401-PadW1) -> /User IO/IO15
- U401 pad W2: /User IO/B1 -> /User IO/IO14
- U401 pad W4: /User IO/IO7 -> /User IO/IO3
- U401 pad W5: /User IO/IO13 -> Net-(U401-PadW5)
- U401 pad W6: /User IO/IO12 -> Net-(U401-PadW6)
- U401 pad Y1: Net-(U401-PadY1) -> /User IO/IO13
- U401 pad Y2: Net-(U401-PadY2) -> /User IO/IO12
- U401 pad Y3: /User IO/IO0 -> /User IO/IO6
- U401 pad Y4: /User IO/IO4 -> /User IO/IO2
Routing:
- net /PCIe Connector/12V_power: track 3.02 -> 91.5 mm, vias 1 -> 3
- net /User IO/B1: track 0.00 -> 45.7 mm
- net /PCIe Connector/PERST#R: track 0.00 -> 44.9 mm, vias 0 -> 3
- net /User IO/IO15: track 0.00 -> 41.6 mm
- net (no net): track 71.1 -> 30.0 mm, vias 0 -> 9
- net +3V3: track 124.8 -> 165.2 mm
- net /User IO/IO13: track 0.00 -> 39.0 mm
- net /User IO/B0: track 0.00 -> 38.6 mm
- net /User IO/IO14: track 0.00 -> 38.6 mm
- net /User IO/IO9: track 0.00 -> 37.9 mm, vias 0 -> 1
- net /User IO/IO11: track 0.00 -> 35.8 mm
- net /User IO/IO12: track 0.00 -> 35.7 mm
- net /User IO/IO8: track 0.00 -> 34.9 mm, vias 0 -> 1
- net /PCIe Connector/PCIE_PRSNT#1: track 0.00 -> 32.6 mm, vias 0 -> 1
- net /User IO/IO10: track 0.00 -> 30.4 mm
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
Commit message: Pending final check
Parts:
- added C312: 47uF, wbraun_smd:C_0805, F.Cu at (64.2, 85.0)
- added C315: 47uF, wbraun_smd:C_0805, F.Cu at (64.2, 89.0)
- added C317: 47uF, wbraun_smd:C_0805, F.Cu at (67.8, 71.8)
- added C318: 47uF, wbraun_smd:C_0805, F.Cu at (67.8, 76.0)
- added C319: 47uF, wbraun_smd:C_0805, F.Cu at (67.0, 85.0)
- added C320: 47uF, wbraun_smd:C_0805, F.Cu at (67.0, 89.0)
- added R309: 215K, wbraun_smd:R_0402, F.Cu at (50.8, 86.2)
- moved C446 3.16 mm to (105.0, 90.0), turned to 0 degrees
- moved C313 1.07 mm to (104.5, 109.7), turned to 0 degrees
- moved R201 0.50 mm to (108.0, 112.5)
- moved C314 0.25 mm to (102.0, 105.8)
Connections:
- net /FPGA Config/FPGA_CLK renamed Net-(U401-PadW19)
Routing:
- net GND: track 326.3 -> 475.9 mm, vias 247 -> 311
- net (no net): track 30.0 -> 0.00 mm, vias 9 -> 0
- net +1V8: track 51.5 -> 65.0 mm, vias 16 -> 18
- net Net-(R309-Pad1): track 0.00 -> 5.92 mm
- net /FPGA Transceivers/SFP_TX_N: track 43.3 -> 47.1 mm
- net /Power Rails/1V8_PGOOD: track 30.8 -> 33.4 mm
- net /FPGA Transceivers/SFP_TX_P: track 44.5 -> 47.1 mm
- net /FPGA Transceivers/PCIE_CLK_N: track 47.0 -> 49.2 mm
- net +3V3: track 165.2 -> 167.3 mm
- net +5V: track 13.1 -> 14.7 mm
- net +12V: track 28.6 -> 27.6 mm, vias 16 -> 15
- net /FPGA Transceivers/PCIE_CLK_P: track 48.8 -> 49.6 mm
- net /FPGA Transceivers/PCIE_TX0_P: track 40.0 -> 40.8 mm
- net /FPGA Power/MGTAVCC: track 7.02 -> 7.66 mm
- net /FPGA Transceivers/PCIE_RX0_P: track 67.0 -> 67.6 mm
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
Commit message: Ready for fab
Parts:
- added REF**: MountingHole_4mm, Mounting_Holes:MountingHole_4mm, F.Cu at (136.0, 46.0)
- added REF**: MountingHole_4mm, Mounting_Holes:MountingHole_4mm, F.Cu at (130.0, 133.0)
- added REF**: MountingHole_3-5mm, Mounting_Holes:MountingHole_3-5mm, F.Cu at (119.5, 47.0)
- added REF**: MountingHole_3-5mm, Mounting_Holes:MountingHole_3-5mm, F.Cu at (79.5, 47.0)
- moved R202 25.5 mm to (84.5, 136.0), turned to 180 degrees
- moved C701 0.25 mm to (81.2, 60.0)
- moved C702 0.25 mm to (81.2, 61.5)
Connections:
- U401 pad AA7: (no net) -> +3V3
Routing:
- net GND: track 475.9 -> 501.9 mm, vias 311 -> 327
- net /PCIe Connector/PCIE_PRSNT#1: track 32.6 -> 52.6 mm
- net /PCIe Connector/PERST#R: track 44.4 -> 49.6 mm
- net /PCIe Connector/CLKREQ#: track 21.5 -> 25.2 mm, vias 2 -> 0
- net /FPGA Transceivers/PCIE_CLK_N: track 49.2 -> 52.6 mm
- net /FPGA Transceivers/SFP_CLK_C_N: track 50.2 -> 47.6 mm
- net /FPGA Transceivers/PCIE_CLK_P: track 49.6 -> 51.7 mm
- net /FPGA Transceivers/SFP_CLK_C_P: track 49.1 -> 47.6 mm
- net /FPGA Transceivers/PCIE_RX0_P: track 67.6 -> 68.9 mm
- net /FPGA Transceivers/PCIE_RX0_N: track 67.6 -> 68.8 mm
- net /FPGA Transceivers/SFP_RX_N: track 49.5 -> 50.7 mm
- net /FPGA Transceivers/SFP_RX_P: track 49.5 -> 50.6 mm
- net /FPGA Transceivers/PCIE_TX0_N: track 40.8 -> 39.9 mm
- net /FPGA Transceivers/SFP_TX_P: track 47.1 -> 47.8 mm
- net /FPGA Transceivers/SFP_TX_N: track 47.1 -> 47.8 mm
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Other:
- board text added: "100 ohm diff: 0.2mm width, 0.13mm spacing 50 ohm SE: 0.35mm"
- board text added: "Artix-7 PCIe Dev Board V1.0 WBRAUN@MIT.EDU"
- board text removed: "100 ohm diff: 0.15mm width, 0.15mm spacing 50 ohm SE: 0.35mm"
- board text removed: "Pin 1 faces in"
