File: pcb/myriadRF_IO.sch (KiCad schematic (older format))
At the start: 2 parts

Commit message: schematic completed. Time for review
Connections:
- net RX_CLK: no longer U?.K18 (IO_L13P_T2_MRCC_15)
- net TX_CLK: no longer U?.J19 (IO_L12P_T1_MRCC_15)
- new net RX_CLK_FPGA: U?.K18 (IO_L13P_T2_MRCC_15)
- new net TX_CLK_FPGA: U?.J19 (IO_L12P_T1_MRCC_15)
Other:
- note added: "80[S] denotes receptacle, this is correct"
Changed lines of the file:
@@
 LIBS:valves
 LIBS:wbraun_ic_lib
-LIBS:xilinx-artix7
-LIBS:FMC_connector-cache
+LIBS:pgmfoot
 LIBS:artix7_pcie_pcb-cache
 EELAYER 25 0
@@
 $Descr A4 11693 8268
 encoding utf-8
-Sheet 8 10
+Sheet 8 12
 Title ""
 Date ""
@@
 TXD11
 Text Label 5550 3500 2    50   ~ 0
-TXCLK
+TXCLK_FPGA
 Text Label 5550 3700 2    50   ~ 0
-RXCLK
+RXCLK_FPGA
 Text Label 5550 3900 2    50   ~ 0
 RXIQSEL
@@
 Text Label 5550 6100 2    50   ~ 0
 RXEN
-Text GLabel 10100 1300 2    50   Input ~ 0
-RF_CLK
-Text GLabel 10100 1500 2    50   Input ~ 0
-TX_CLK
-Text GLabel 10100 1700 2    50   Input ~ 0
-RX_CLK
 Wire Wire Line
 	10100 1300 9700 1300
@@
 Text Label 9700 1700 2    50   ~ 0
 RXCLK
+Text HLabel 10100 1300 2    60   Input ~ 0
+RF_CLK
+Text HLabel 10100 1500 2    60   Input ~ 0
+TX_CLK
+Text HLabel 10100 1700 2    60   Input ~ 0
+RX_CLK
+Text Notes 2100 7150 0    60   ~ 0
+80[S] denotes receptacle, this is correct
+Wire Wire Line
+	9700 1900 10100 1900
+Text Label 9700 1900 2    60   ~ 0
+TXCLK_FPGA
+Text HLabel 10100 1900 2    60   Input ~ 0
+TX_CLK_FPGA
+Wire Wire Line
+	9700 2100 10100 2100
+Text Label 9700 2100 2    60   ~ 0
+RXCLK_FPGA
+Text HLabel 10100 2100 2    60   Input ~ 0
+RX_CLK_FPGA
 $EndSCHEMATC

Commit message: Added part numbers and updated schematic
Parts:
- gave numbers to parts that had none: 2
Changed lines of the file:
@@
 $EndDescr
 $Comp
-L FX10B-80S/8-SV J?
+L FX10B-80S/8-SV J801
 U 1 1 5633F39C
 P 3000 4100
-F 0 "J?" H 3350 6950 60  0000 C CNN
+F 0 "J801" H 3350 6950 60  0000 C CNN
 F 1 "FX10B-80S/8-SV" H 2800 1200 60  0000 C CNN
 F 2 "" H 3000 4100 60  0000 C CNN
@@
 $EndComp
 $Comp
-L +3V3 #PWR?
+L +3V3 #PWR816
 U 1 1 5633FA2D
 P 1900 2000
-F 0 "#PWR?" H 1900 1850 50  0001 C CNN
+F 0 "#PWR816" H 1900 1850 50  0001 C CNN
 F 1 "+3V3" H 1900 2140 50  0000 C CNN
 F 2 "" H 1900 2000 60  0000 C CNN
@@
 $EndComp
 $Comp
-L +3V3 #PWR?
+L +3V3 #PWR819
 U 1 1 5633FA45
 P 4100 2000
-F 0 "#PWR?" H 4100 1850 50  0001 C CNN
+F 0 "#PWR819" H 4100 1850 50  0001 C CNN
 F 1 "+3V3" H 4100 2140 50  0000 C CNN
 F 2 "" H 4100 2000 60  0000 C CNN
@@
 $EndComp
 $Comp
-L GND #PWR?
+L GND #PWR801
 U 1 1 5633FAA5
 P 1700 1800
-F 0 "#PWR?" H 1700 1550 50  0001 C CNN
+F 0 "#PWR801" H 1700 1550 50  0001 C CNN
 F 1 "GND" H 1700 1650 50  0000 C CNN
 F 2 "" H 1700 1800 60  0000 C CNN
@@
 $EndComp
 $Comp
-L GND #PWR?
+L GND #PWR820
 U 1 1 5633FABD
 P 4400 1800
-F 0 "#PWR?" H 4400 1550 50  0001 C CNN
+F 0 "#PWR820" H 4400 1550 50  0001 C CNN
 F 1 "GND" H 4400 1650 50  0000 C CNN
 F 2 "" H 4400 1800 60  0000 C CNN
@@
 $EndComp
 $Comp
-L +5V #PWR?
+L +5V #PWR817
 U 1 1 5633FAF5
 P 2000 1500
-F 0 "#PWR?" H 2000 1350 50  0001 C CNN
+F 0 "#PWR817" H 2000 1350 50  0001 C CNN
 F 1 "+5V" H 2000 1640 50  0000 C CNN
 F 2 "" H 2000 1500 60  0000 C CNN
@@
 $EndComp
 $Comp
-L +5V #PWR?
+L +5V #PWR818
 U 1 1 5633FB0D
 P 4000 1500
-F 0 "#PWR?" H 4000 1350 50  0001 C CNN
+F 0 "#PWR818" H 4000 1350 50  0001 C CNN
 F 1 "+5V" H 4000 1640 50  0000 C CNN
 F 2 "" H 4000 1500 60  0000 C CNN
@@
 $EndComp
 $Comp
-L GND #PWR?
+L GND #PWR803
 U 1 1 5633FBA6
 P 1700 2400
-F 0 "#PWR?" H 1700 2150 50  0001 C CNN
+F 0 "#PWR803" H 1700 2150 50  0001 C CNN
 F 1 "GND" H 1700 2250 50  0000 C CNN
 F 2 "" H 1700 2400 60  0000 C CNN
@@
 $EndComp
 $Comp
-L GND #PWR?
+L GND #PWR822
 U 1 1 5633FBBE
 P 4400 2400
-F 0 "#PWR?" H 4400 2150 50  0001 C CNN
+F 0 "#PWR822" H 4400 2150 50  0001 C CNN
 F 1 "GND" H 4400 2250 50  0000 C CNN
 F 2 "" H 4400 2400 60  0000 C CNN
@@
 $EndComp
 $Comp
-L GND #PWR?
+L GND #PWR804
 U 1 1 5633FC09
 P 1700 2700
-F 0 "#PWR?" H 1700 2450 50  0001 C CNN
+F 0 "#PWR804" H 1700 2450 50  0001 C CNN
 F 1 "GND" H 1700 2550 50  0000 C CNN
 F 2 "" H 1700 2700 60  0000 C CNN
@@
 $EndComp
 $Comp
-L GND #PWR?
+L GND #PWR823
 U 1 1 5633FC21
 P 4400 2700
-F 0 "#PWR?" H 4400 2450 50  0001 C CNN
+F 0 "#PWR823" H 4400 2450 50  0001 C CNN
 F 1 "GND" H 4400 2550 50  0000 C CNN
 F 2 "" H 4400 2700 60  0000 C CNN
@@
 RXEN
 $Comp
-L GND #PWR?
+L GND #PWR805
 U 1 1 56340878
 P 1700 3200
-F 0 "#PWR?" H 1700 2950 50  0001 C CNN
+F 0 "#PWR805" H 1700 2950 50  0001 C CNN
 F 1 "GND" H 1700 3050 50  0000 C CNN
 F 2 "" H 1700 3200 60  0000 C CNN
@@
 $EndComp
 $Comp
-L GND #PWR?
+L GND #PWR807
 U 1 1 5634089E
 P 1700 4000
-F 0 "#PWR?" H 1700 3750 50  0001 C CNN
+F 0 "#PWR807" H 1700 3750 50  0001 C CNN
 F 1 "GND" H 1700 3850 50  0000 C CNN
 F 2 "" H 1700 4000 60  0000 C CNN
@@
 $EndComp
 $Comp
-L GND #PWR?
+L GND #PWR808
 U 1 1 563408B6
 P 1700 4500
-F 0 "#PWR?" H 1700 4250 50  0001 C CNN
+F 0 "#PWR808" H 1700 4250 50  0001 C CNN
 F 1 "GND" H 1700 4350 50  0000 C CNN
 F 2 "" H 1700 4500 60  0000 C CNN
@@
 $EndComp
 $Comp
-L GND #PWR?
+L GND #PWR810
 U 1 1 563408CE
 P 1700 5300
-F 0 "#PWR?" H 1700 5050 50  0001 C CNN
+F 0 "#PWR810" H 1700 5050 50  0001 C CNN
 F 1 "GND" H 1700 5150 50  0000 C CNN
 F 2 "" H 1700 5300 60  0000 C CNN
@@
 $EndComp
 $Comp
-L GND #PWR?
+L GND #PWR811
 U 1 1 563408E6
 P 1700 5600
-F 0 "#PWR?" H 1700 5350 50  0001 C CNN
+F 0 "#PWR811" H 1700 5350 50  0001 C CNN
 F 1 "GND" H 1700 5450 50  0000 C CNN
 F 2 "" H 1700 5600 60  0000 C CNN
@@
 $EndComp
 $Comp
-L GND #PWR?
+L GND #PWR824
 U 1 1 563408FE
 P 4400 3200
-F 0 "#PWR?" H 4400 2950 50  0001 C CNN
+F 0 "#PWR824" H 4400 2950 50  0001 C CNN
 F 1 "GND" H 4400 3050 50  0000 C CNN
 F 2 "" H 4400 3200 60  0000 C CNN
@@
 $EndComp
 $Comp
-L GND #PWR?
+L GND #PWR826
 U 1 1 56340916
 P 4400 4000
-F 0 "#PWR?" H 4400 3750 50  0001 C CNN
+F 0 "#PWR826" H 4400 3750 50  0001 C CNN
 F 1 "GND" H 4400 3850 50  0000 C CNN
 F 2 "" H 4400 4000 60  0000 C CNN
@@
 $EndComp
 $Comp
-L GND #PWR?
+L GND #PWR827
 U 1 1 5634092E
 P 4400 4500
-F 0 "#PWR?" H 4400 4250 50  0001 C CNN
+F 0 "#PWR827" H 4400 4250 50  0001 C CNN
 F 1 "GND" H 4400 4350 50  0000 C CNN
 F 2 "" H 4400 4500 60  0000 C CNN
@@
 $EndComp
 $Comp
-L GND #PWR?
+L GND #PWR829
 U 1 1 56340946
 P 4400 5300
-F 0 "#PWR?" H 4400 5050 50  0001 C CNN
+F 0 "#PWR829" H 4400 5050 50  0001 C CNN
 F 1 "GND" H 4400 5150 50  0000 C CNN
 F 2 "" H 4400 5300 60  0000 C CNN
@@
 $EndComp
 $Comp
-L GND #PWR?
+L GND #PWR830
 U 1 1 5634095E
 P 4400 5600
-F 0 "#PWR?" H 4400 5350 50  0001 C CNN
+F 0 "#PWR830" H 4400 5350 50  0001 C CNN
 F 1 "GND" H 4400 5450 50  0000 C CNN
 F 2 "" H 4400 5600 60  0000 C CNN
@@
 $EndComp
 $Comp
-L GND #PWR?
+L GND #PWR813
 U 1 1 5634099A
 P 1700 6400
-F 0 "#PWR?" H 1700 6150 50  0001 C CNN
+F 0 "#PWR813" H 1700 6150 50  0001 C CNN
 F 1 "GND" H 1700 6250 50  0000 C CNN
 F 2 "" H 1700 6400 60  0000 C CNN
@@
 $EndComp
 $Comp
-L GND #PWR?
+L GND #PWR814
 U 1 1 563409B2
 P 1700 6600
-F 0 "#PWR?" H 1700 6350 50  0001 C CNN
+F 0 "#PWR814" H 1700 6350 50  0001 C CNN
 F 1 "GND" H 1700 6450 50  0000 C CNN
 F 2 "" H 1700 6600 60  0000 C CNN
@@
 $EndComp
 $Comp
-L GND #PWR?
+L GND #PWR821
 U 1 1 563415C5
 P 4400 2200
-F 0 "#PWR?" H 4400 1950 50  0001 C CNN
+F 0 "#PWR821" H 4400 1950 50  0001 C CNN
 F 1 "GND" H 4400 2050 50  0000 C CNN
 F 2 "" H 4400 2200 60  0000 C CNN
@@
 $EndComp
 $Comp
-L GND #PWR?
+L GND #PWR802
 U 1 1 563415E1
 P 1700 2200
-F 0 "#PWR?" H 1700 1950 50  0001 C CNN
+F 0 "#PWR802" H 1700 1950 50  0001 C CNN
 F 1 "GND" H 1700 2050 50  0000 C CNN
 F 2 "" H 1700 2200 60  0000 C CNN
@@
 $EndComp
 $Comp
-L GND #PWR?
+L GND #PWR806
 U 1 1 563415F9
 P 1700 3500
-F 0 "#PWR?" H 1700 3250 50  0001 C CNN
+F 0 "#PWR806" H 1700 3250 50  0001 C CNN
 F 1 "GND" H 1700 3350 50  0000 C CNN
 F 2 "" H 1700 3500 60  0000 C CNN
@@
 $EndComp
 $Comp
-L GND #PWR?
+L GND #PWR825
 U 1 1 56341611
 P 4400 3500
-F 0 "#PWR?" H 4400 3250 50  0001 C CNN
+F 0 "#PWR825" H 4400 3250 50  0001 C CNN
 F 1 "GND" H 4400 3350 50  0000 C CNN
 F 2 "" H 4400 3500 60  0000 C CNN
@@
 $EndComp
 $Comp
-L GND #PWR?
+L GND #PWR828
 U 1 1 56341635
 P 4400 4800
-F 0 "#PWR?" H 4400 4550 50  0001 C CNN
+F 0 "#PWR828" H 4400 4550 50  0001 C CNN
 F 1 "GND" H 4400 4650 50  0000 C CNN
 F 2 "" H 4400 4800 60  0000 C CNN
@@
 $EndComp
 $Comp
-L GND #PWR?
+L GND #PWR809
 U 1 1 5634164D
 P 1700 4800
-F 0 "#PWR?" H 1700 4550 50  0001 C CNN
+F 0 "#PWR809" H 1700 4550 50  0001 C CNN
 F 1 "GND" H 1700 4650 50  0000 C CNN
 F 2 "" H 1700 4800 60  0000 C CNN
@@
 $EndComp
 $Comp
-L GND #PWR?
+L GND #PWR831
 U 1 1 56341671
 P 4400 6100
-F 0 "#PWR?" H 4400 5850 50  0001 C CNN
+F 0 "#PWR831" H 4400 5850 50  0001 C CNN
 F 1 "GND" H 4400 5950 50  0000 C CNN
 F 2 "" H 4400 6100 60  0000 C CNN
@@
 $EndComp
 $Comp
-L GND #PWR?
+L GND #PWR812
 U 1 1 56341689
 P 1700 6100
-F 0 "#PWR?" H 1700 5850 50  0001 C CNN
+F 0 "#PWR812" H 1700 5850 50  0001 C CNN
 F 1 "GND" H 1700 5950 50  0000 C CNN
 F 2 "" H 1700 6100 60  0000 C CNN
@@
 $EndComp
 $Comp
-L GND #PWR?
+L GND #PWR832
 U 1 1 563416A1
 P 4400 6800
-F 0 "#PWR?" H 4400 6550 50  0001 C CNN
+F 0 "#PWR832" H 4400 6550 50  0001 C CNN
 F 1 "GND" H 4400 6650 50  0000 C CNN
 F 2 "" H 4400 6800 60  0000 C CNN
@@
 $EndComp
 $Comp
-L GND #PWR?
+L GND #PWR815
 U 1 1 563416B9
 P 1700 6800
-F 0 "#PWR?" H 1700 6550 50  0001 C CNN
+F 0 "#PWR815" H 1700 6550 50  0001 C CNN
 F 1 "GND" H 1700 6650 50  0000 C CNN
 F 2 "" H 1700 6800 60  0000 C CNN
@@
 $EndComp
 $Comp
-L XC7Axxt-FGG484 U?
+L XC7Axxt-FGG484 U401
 U 3 1 56341B2F
 P 6950 3650
-F 0 "U?" H 6050 1050 60  0000 C CNN
+F 0 "U401" H 6050 1050 60  0000 C CNN
 F 1 "XC7Axxt-FGG484" H 6350 6250 60  0000 C CNN
 F 2 "" H 6950 3700 60  0000 C CNN

Commit message: mostly done with component placement
Parts:
- J801: footprint (none) -> wbraun_smd:FX10B_80S_8_SV
- U401: footprint (none) -> wbraun_smd:BGA_484_22x22_FULLARRAY_1MM
Changed lines of the file:
@@
 F 0 "J801" H 3350 6950 60  0000 C CNN
 F 1 "FX10B-80S/8-SV" H 2800 1200 60  0000 C CNN
-F 2 "" H 3000 4100 60  0000 C CNN
+F 2 "wbraun_smd:FX10B_80S_8_SV" H 3000 4100 60  0001 C CNN
 F 3 "" H 3000 4100 60  0000 C CNN
 	1    3000 4100
@@
 $EndComp
 $Comp
-L +3V3 #PWR816
+L +3V3 #PWR089
 U 1 1 5633FA2D
 P 1900 2000
-F 0 "#PWR816" H 1900 1850 50  0001 C CNN
+F 0 "#PWR089" H 1900 1850 50  0001 C CNN
 F 1 "+3V3" H 1900 2140 50  0000 C CNN
 F 2 "" H 1900 2000 60  0000 C CNN
@@
 $EndComp
 $Comp
-L +3V3 #PWR819
+L +3V3 #PWR090
 U 1 1 5633FA45
 P 4100 2000
-F 0 "#PWR819" H 4100 1850 50  0001 C CNN
+F 0 "#PWR090" H 4100 1850 50  0001 C CNN
 F 1 "+3V3" H 4100 2140 50  0000 C CNN
 F 2 "" H 4100 2000 60  0000 C CNN
@@
 $EndComp
 $Comp
-L GND #PWR801
+L GND #PWR091
 U 1 1 5633FAA5
 P 1700 1800
-F 0 "#PWR801" H 1700 1550 50  0001 C CNN
+F 0 "#PWR091" H 1700 1550 50  0001 C CNN
 F 1 "GND" H 1700 1650 50  0000 C CNN
 F 2 "" H 1700 1800 60  0000 C CNN
@@
 $EndComp
 $Comp
-L GND #PWR820
+L GND #PWR092
 U 1 1 5633FABD
 P 4400 1800
-F 0 "#PWR820" H 4400 1550 50  0001 C CNN
+F 0 "#PWR092" H 4400 1550 50  0001 C CNN
 F 1 "GND" H 4400 1650 50  0000 C CNN
 F 2 "" H 4400 1800 60  0000 C CNN
@@
 $EndComp
 $Comp
-L +5V #PWR817
+L +5V #PWR093
 U 1 1 5633FAF5
 P 2000 1500
-F 0 "#PWR817" H 2000 1350 50  0001 C CNN
+F 0 "#PWR093" H 2000 1350 50  0001 C CNN
 F 1 "+5V" H 2000 1640 50  0000 C CNN
 F 2 "" H 2000 1500 60  0000 C CNN
@@
 $EndComp
 $Comp
-L +5V #PWR818
+L +5V #PWR094
 U 1 1 5633FB0D
 P 4000 1500
-F 0 "#PWR818" H 4000 1350 50  0001 C CNN
+F 0 "#PWR094" H 4000 1350 50  0001 C CNN
 F 1 "+5V" H 4000 1640 50  0000 C CNN
 F 2 "" H 4000 1500 60  0000 C CNN
@@
 $EndComp
 $Comp
-L GND #PWR803
+L GND #PWR095
 U 1 1 5633FBA6
 P 1700 2400
-F 0 "#PWR803" H 1700 2150 50  0001 C CNN
+F 0 "#PWR095" H 1700 2150 50  0001 C CNN
 F 1 "GND" H 1700 2250 50  0000 C CNN
 F 2 "" H 1700 2400 60  0000 C CNN
@@
 $EndComp
 $Comp
-L GND #PWR822
+L GND #PWR096
 U 1 1 5633FBBE
 P 4400 2400
-F 0 "#PWR822" H 4400 2150 50  0001 C CNN
+F 0 "#PWR096" H 4400 2150 50  0001 C CNN
 F 1 "GND" H 4400 2250 50  0000 C CNN
 F 2 "" H 4400 2400 60  0000 C CNN
@@
 $EndComp
 $Comp
-L GND #PWR804
+L GND #PWR097
 U 1 1 5633FC09
 P 1700 2700
-F 0 "#PWR804" H 1700 2450 50  0001 C CNN
+F 0 "#PWR097" H 1700 2450 50  0001 C CNN
 F 1 "GND" H 1700 2550 50  0000 C CNN
 F 2 "" H 1700 2700 60  0000 C CNN
@@
 $EndComp
 $Comp
-L GND #PWR823
+L GND #PWR098
 U 1 1 5633FC21
 P 4400 2700
-F 0 "#PWR823" H 4400 2450 50  0001 C CNN
+F 0 "#PWR098" H 4400 2450 50  0001 C CNN
 F 1 "GND" H 4400 2550 50  0000 C CNN
 F 2 "" H 4400 2700 60  0000 C CNN
@@
 RXEN
 $Comp
-L GND #PWR805
+L GND #PWR099
 U 1 1 56340878
 P 1700 3200
-F 0 "#PWR805" H 1700 2950 50  0001 C CNN
+F 0 "#PWR099" H 1700 2950 50  0001 C CNN
 F 1 "GND" H 1700 3050 50  0000 C CNN
 F 2 "" H 1700 3200 60  0000 C CNN
@@
 $EndComp
 $Comp
-L GND #PWR807
+L GND #PWR0100
 U 1 1 5634089E
 P 1700 4000
-F 0 "#PWR807" H 1700 3750 50  0001 C CNN
+F 0 "#PWR0100" H 1700 3750 50  0001 C CNN
 F 1 "GND" H 1700 3850 50  0000 C CNN
 F 2 "" H 1700 4000 60  0000 C CNN
@@
 $EndComp
 $Comp
-L GND #PWR808
+L GND #PWR0101
 U 1 1 563408B6
 P 1700 4500
-F 0 "#PWR808" H 1700 4250 50  0001 C CNN
+F 0 "#PWR0101" H 1700 4250 50  0001 C CNN
 F 1 "GND" H 1700 4350 50  0000 C CNN
 F 2 "" H 1700 4500 60  0000 C CNN
@@
 $EndComp
 $Comp
-L GND #PWR810
+L GND #PWR0102
 U 1 1 563408CE
 P 1700 5300
-F 0 "#PWR810" H 1700 5050 50  0001 C CNN
+F 0 "#PWR0102" H 1700 5050 50  0001 C CNN
 F 1 "GND" H 1700 5150 50  0000 C CNN
 F 2 "" H 1700 5300 60  0000 C CNN
@@
 $EndComp
 $Comp
-L GND #PWR811
+L GND #PWR0103
 U 1 1 563408E6
 P 1700 5600
-F 0 "#PWR811" H 1700 5350 50  0001 C CNN
+F 0 "#PWR0103" H 1700 5350 50  0001 C CNN
 F 1 "GND" H 1700 5450 50  0000 C CNN
 F 2 "" H 1700 5600 60  0000 C CNN
@@
 $EndComp
 $Comp
-L GND #PWR824
+L GND #PWR0104
 U 1 1 563408FE
 P 4400 3200
-F 0 "#PWR824" H 4400 2950 50  0001 C CNN
+F 0 "#PWR0104" H 4400 2950 50  0001 C CNN
 F 1 "GND" H 4400 3050 50  0000 C CNN
 F 2 "" H 4400 3200 60  0000 C CNN
@@
 $EndComp
 $Comp
-L GND #PWR826
+L GND #PWR0105
 U 1 1 56340916
 P 4400 4000
-F 0 "#PWR826" H 4400 3750 50  0001 C CNN
+F 0 "#PWR0105" H 4400 3750 50  0001 C CNN
 F 1 "GND" H 4400 3850 50  0000 C CNN
 F 2 "" H 4400 4000 60  0000 C CNN
@@
 $EndComp
 $Comp
-L GND #PWR827
+L GND #PWR0106
 U 1 1 5634092E
 P 4400 4500
-F 0 "#PWR827" H 4400 4250 50  0001 C CNN
+F 0 "#PWR0106" H 4400 4250 50  0001 C CNN
 F 1 "GND" H 4400 4350 50  0000 C CNN
 F 2 "" H 4400 4500 60  0000 C CNN
@@
 $EndComp
 $Comp
-L GND #PWR829
+L GND #PWR0107
 U 1 1 56340946
 P 4400 5300
-F 0 "#PWR829" H 4400 5050 50  0001 C CNN
+F 0 "#PWR0107" H 4400 5050 50  0001 C CNN
 F 1 "GND" H 4400 5150 50  0000 C CNN
 F 2 "" H 4400 5300 60  0000 C CNN
@@
 $EndComp
 $Comp
-L GND #PWR830
+L GND #PWR0108
 U 1 1 5634095E
 P 4400 5600
-F 0 "#PWR830" H 4400 5350 50  0001 C CNN
+F 0 "#PWR0108" H 4400 5350 50  0001 C CNN
 F 1 "GND" H 4400 5450 50  0000 C CNN
 F 2 "" H 4400 5600 60  0000 C CNN
@@
 $EndComp
 $Comp
-L GND #PWR813
+L GND #PWR0109
 U 1 1 5634099A
 P 1700 6400
-F 0 "#PWR813" H 1700 6150 50  0001 C CNN
+F 0 "#PWR0109" H 1700 6150 50  0001 C CNN
 F 1 "GND" H 1700 6250 50  0000 C CNN
 F 2 "" H 1700 6400 60  0000 C CNN
@@
 $EndComp
 $Comp
-L GND #PWR814
+L GND #PWR0110
 U 1 1 563409B2
 P 1700 6600
-F 0 "#PWR814" H 1700 6350 50  0001 C CNN
+F 0 "#PWR0110" H 1700 6350 50  0001 C CNN
 F 1 "GND" H 1700 6450 50  0000 C CNN
 F 2 "" H 1700 6600 60  0000 C CNN
@@
 $EndComp
 $Comp
-L GND #PWR821
+L GND #PWR0111
 U 1 1 563415C5
 P 4400 2200
-F 0 "#PWR821" H 4400 1950 50  0001 C CNN
+F 0 "#PWR0111" H 4400 1950 50  0001 C CNN
 F 1 "GND" H 4400 2050 50  0000 C CNN
 F 2 "" H 4400 2200 60  0000 C CNN
@@
 $EndComp
 $Comp
-L GND #PWR802
+L GND #PWR0112
 U 1 1 563415E1
 P 1700 2200
-F 0 "#PWR802" H 1700 1950 50  0001 C CNN
+F 0 "#PWR0112" H 1700 1950 50  0001 C CNN
 F 1 "GND" H 1700 2050 50  0000 C CNN
 F 2 "" H 1700 2200 60  0000 C CNN
@@
 $EndComp
 $Comp
-L GND #PWR806
+L GND #PWR0113
 U 1 1 563415F9
 P 1700 3500
-F 0 "#PWR806" H 1700 3250 50  0001 C CNN
+F 0 "#PWR0113" H 1700 3250 50  0001 C CNN
 F 1 "GND" H 1700 3350 50  0000 C CNN
 F 2 "" H 1700 3500 60  0000 C CNN
@@
 $EndComp
 $Comp
-L GND #PWR825
+L GND #PWR0114
 U 1 1 56341611
 P 4400 3500
-F 0 "#PWR825" H 4400 3250 50  0001 C CNN
+F 0 "#PWR0114" H 4400 3250 50  0001 C CNN
 F 1 "GND" H 4400 3350 50  0000 C CNN
 F 2 "" H 4400 3500 60  0000 C CNN
@@
 $EndComp
 $Comp
-L GND #PWR828
+L GND #PWR0115
 U 1 1 56341635
 P 4400 4800
-F 0 "#PWR828" H 4400 4550 50  0001 C CNN
+F 0 "#PWR0115" H 4400 4550 50  0001 C CNN
 F 1 "GND" H 4400 4650 50  0000 C CNN
 F 2 "" H 4400 4800 60  0000 C CNN
@@
 $EndComp
 $Comp
-L GND #PWR809
+L GND #PWR0116
 U 1 1 5634164D
 P 1700 4800
-F 0 "#PWR809" H 1700 4550 50  0001 C CNN
+F 0 "#PWR0116" H 1700 4550 50  0001 C CNN
 F 1 "GND" H 1700 4650 50  0000 C CNN
 F 2 "" H 1700 4800 60  0000 C CNN
@@
 $EndComp
 $Comp
-L GND #PWR831
+L GND #PWR0117
 U 1 1 56341671
 P 4400 6100
-F 0 "#PWR831" H 4400 5850 50  0001 C CNN
+F 0 "#PWR0117" H 4400 5850 50  0001 C CNN
 F 1 "GND" H 4400 5950 50  0000 C CNN
 F 2 "" H 4400 6100 60  0000 C CNN
@@
 $EndComp
 $Comp
-L GND #PWR812
+L GND #PWR0118
 U 1 1 56341689
 P 1700 6100
-F 0 "#PWR812" H 1700 5850 50  0001 C CNN
+F 0 "#PWR0118" H 1700 5850 50  0001 C CNN
 F 1 "GND" H 1700 5950 50  0000 C CNN
 F 2 "" H 1700 6100 60  0000 C CNN
@@
 $EndComp
 $Comp
-L GND #PWR832
+L GND #PWR0119
 U 1 1 563416A1
 P 4400 6800
-F 0 "#PWR832" H 4400 6550 50  0001 C CNN
+F 0 "#PWR0119" H 4400 6550 50  0001 C CNN
 F 1 "GND" H 4400 6650 50  0000 C CNN
 F 2 "" H 4400 6800 60  0000 C CNN
@@
 $EndComp
 $Comp
-L GND #PWR815
+L GND #PWR0120
 U 1 1 563416B9
 P 1700 6800
-F 0 "#PWR815" H 1700 6550 50  0001 C CNN
+F 0 "#PWR0120" H 1700 6550 50  0001 C CNN
 F 1 "GND" H 1700 6650 50  0000 C CNN
 F 2 "" H 1700 6800 60  0000 C CNN
@@
 F 0 "U401" H 6050 1050 60  0000 C CNN
 F 1 "XC7Axxt-FGG484" H 6350 6250 60  0000 C CNN
-F 2 "" H 6950 3700 60  0000 C CNN
+F 2 "wbraun_smd:BGA_484_22x22_FULLARRAY_1MM" H 6950 3700 60  0001 C CNN
 F 3 "" H 6950 3700 60  0000 C CNN
 	3    6950 3650
